File: pcb/can_bus.kicad_sch (KiCad schematic)
At the start: 0 parts

Commit message: Sch almost done, maybe add current sense
Parts:
- added C32, C33, C35: 100n, Capacitor_SMD:C_0603_1608Metric_Pad1.08x0.95mm_HandSolder, symbol Device:C
- added C34: 10u, Capacitor_SMD:C_1206_3216Metric_Pad1.33x1.80mm_HandSolder, symbol Device:C
- added C39, C40, C41: 4.7pF, Capacitor_SMD:C_0603_1608Metric_Pad1.08x0.95mm_HandSolder, symbol Device:C
- added IC2: ATA6561-GAQW-N, SOIC127P600X175-8N, symbol SamacSys_Parts:ATA6561-GAQW-N
- added Q2: BSS138, Package_TO_SOT_SMD:SOT-23, symbol Transistor_FET:BSS138
- added R21, R22: 59, Resistor_SMD:R_0603_1608Metric_Pad0.98x0.95mm_HandSolder, symbol Device:R
- added R23: 560R, Resistor_SMD:R_0603_1608Metric_Pad0.98x0.95mm_HandSolder, symbol Device:R
- added R24: 100k, Resistor_SMD:R_0603_1608Metric_Pad0.98x0.95mm_HandSolder, symbol Device:R
- added TP10, TP9: TestPoint, TestPoint:TestPoint_Pad_D1.0mm, symbol Connector:TestPoint
- added U701, U702: GAQY212GS, Package_SO:SOP-4_3.8x4.1mm_P2.54mm, symbol Relay_SolidState:CPC1006N
Connections:
- new net: R22.2, U702.3
- new net: C39.1, U701.3, U702.4
- new net: R21.2, U701.4
- new net: R23.2, U701.1
- new net: U701.2, U702.1
- new net: Q2.3 (D), U702.2
- new net +3.3V: C32.1, C33.1, IC2.5 (VIO)
- new net +5V: C34.1, C35.1, IC2.3 (VCC), R23.1
- new net CAN_H: C41.1, IC2.7 (CANH), R22.1
- new net CAN_L: C40.1, IC2.6 (CANL), R21.1
- new net CAN_RX: IC2.4 (RXD), TP10.1
- new net CAN_R_CTRL: Q2.1 (G), R24.1
- new net CAN_STBY: IC2.8 (STBY)
- new net CAN_TX: IC2.1 (TXD), TP9.1
- new net GND: C32.2, C33.2, C34.2, C35.2, C39.2, C40.2, C41.2, IC2.2 (GND), Q2.2 (S), R24.2

Commit message: Scheamtic almost finished, astarted firmware and pcb
Parts:
- C39: value 4.7pF -> 4.7nF
Changed lines of the file:
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@@
 	)
 	(hierarchical_label "CAN_H"
-		(shape input)
+		(shape bidirectional)
 		(at 205.74 77.47 0)
 		(effects
@@
 	)
 	(hierarchical_label "CAN_L"
-		(shape input)
+		(shape bidirectional)
 		(at 205.74 80.01 0)
 		(effects
@@
 	)
 	(hierarchical_label "CAN_RX"
-		(shape input)
+		(shape output)
 		(at 102.87 80.01 180)
 		(effects
@@
 			)
 		)
-		(property "Value" "4.7pF"
+		(property "Value" "4.7nF"
 			(at 189.23 133.3499 0)
 			(show_name no)

Commit message: Schematic finished, first routing
Parts:
- IC2: footprint SOIC127P600X175-8N -> SamacSys_Parts:SOIC127P600X175-8N
Changed lines of the file:
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@@
 			)
 		)
-		(property "Footprint" "SOIC127P600X175-8N"
+		(property "Footprint" "SamacSys_Parts:SOIC127P600X175-8N"
 			(at 137.16 169.85 0)
 			(hide yes)

Commit message: Routing almost finished
Parts:
- removed TP10, TP9: TestPoint, TestPoint:TestPoint_Pad_D1.0mm, symbol Connector:TestPoint

Commit message: Cleaning
Parts:
- Q2: Manufacturer_Part_Number (none) -> BSS138
Changed lines of the file:
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@@
+			)
+		)
+		(property "Manufacturer_Part_Number" "BSS138"
+			(at 156.21 148.59 0)
+			(hide yes)
+			(show_name no)
+			(do_not_autoplace no)
+			(effects
+				(font
+					(size 1.27 1.27)
+				)
 			)
 		)
