File: pcb/geiger_probe.kicad_pcb (KiCad board)
At the start: 2 copper layers, 103 parts, among them J1 Conn_01x05_Pin, J2 TC2030, Q1 DMN3404L, Q2 BSS138, U1 STM32L432KCUx, U2 MCP1700x-330xxMB, U701 GAQY212GS, U702 GAQY212GS, Y1 32,768kHz

Commit message: Schematic finished, first routing
Parts:
- added BT1: MS621FE-FL11E, lib_local:BAT_MS621FE-FL11E, F.Cu at (-29.9, -39.9)
- added C44: 1n, Capacitor_SMD:C_0603_1608Metric, F.Cu at (100.7, -47.6)
- added D5: SMBJ33CA, Diode_SMD:D_SMB, F.Cu at (135.9, 72.2)
- added F2: 01020071Z, SamacSys_Parts:01020071Z, B.Cu at (251.2, 76.7)
- added F3: 01020071Z, SamacSys_Parts:01020071Z, B.Cu at (140.9, 76.7)
- added FL1: ACT45B-510-2P-TL003, SamacSys_Parts:ACT45B1012PTL003, F.Cu at (142.1, 87.7)
- added GD1: 3R090-5S, SamacSys_Parts:3R090A5S, F.Cu at (130.3, 70.9)
- added GD2: 3R090-5S, SamacSys_Parts:3R090A5S, F.Cu at (130.3, 83.3)
- added IC1: LT8606IDC#TRPBF, SamacSys_Parts:SON45P200X200X80-9N-D, F.Cu at (164.6, -31.1)
- added IC2: ATA6561-GAQW-N, SamacSys_Parts:SOIC127P600X175-8N, F.Cu at (-1.80, -57.8)
- added IC8: MCP79410T-I_MS, SamacSys_Parts:SOP65P490X110-8N, F.Cu at (-19.3, -41.8)
- added R28: 1k, Resistor_SMD:R_0603_1608Metric, F.Cu at (104.7, -40.0)
- added U3: INA186A4IDCKR, lib_local:SOT65P210X110-6N, F.Cu at (93.5, -43.4)
- ANODE1, CATHODE1: moved to B.Cu
- J1: value Conn_01x05_Pin -> Conn_01x05_Socket; footprint Connector_PinHeader_2.00mm:PinHeader_1x05_P2.00mm_Vertical -> Connector_PinHeader_2.54mm:PinHeader_1x05_P2.54mm_Vertical
- moved ANODE1 278.7 mm to (255.1, 76.7)
- moved CATHODE1 190.9 mm to (144.8, 76.7)
- moved R15 164.9 mm to (147.1, 87.4), turned to 90 degrees
- moved D6 158.3 mm to (142.9, 70.3), turned to -90 degrees
- moved D8 157.5 mm to (147.4, 70.3), turned to -90 degrees
- moved R16 157.4 mm to (144.4, 82.8), turned to 90 degrees
- moved D9 150.1 mm to (140.6, 83.3), turned to 180 degrees
- moved FB2 148.8 mm to (139.4, 72.8), turned to 90 degrees
- moved FB1 146.9 mm to (139.4, 66.8), turned to 90 degrees
- moved C23 146.9 mm to (156.2, -74.4)
- moved C24 146.9 mm to (156.2, -71.9)
- moved C25 146.9 mm to (156.2, -69.4)
- moved C26 146.9 mm to (156.2, -66.9)
- moved U2 146.9 mm to (153.6, -62.5)
- moved F1 145.0 mm to (135.8, 67.2)
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Connections:
- J1 pad 3: Net-(D9-A2) -> Earth
- J1 pad 4: Net-(D9-A1) -> Net-(D9-A2)
- J1 pad 5: Earth -> Net-(D9-A1)
Routing:
- net Net-(D9-A2): track 0.00 -> 28.4 mm, vias 0 -> 2
- net Net-(D9-A1): track 0.00 -> 25.9 mm
- net Net-(D5-A1): track 0.00 -> 15.3 mm
- net Net-(J1-Pin_1): track 0.00 -> 13.6 mm
- net Net-(D6-K): track 0.00 -> 7.83 mm
- net Net-(D5-A2): track 0.00 -> 7.62 mm
- net Earth: track 0.00 -> 3.99 mm, vias 0 -> 18
- net /PROTECTION/V_zas: track 0.00 -> 3.12 mm
- net Net-(FL1-Pad3): track 0.00 -> 2.65 mm
- net Net-(FL1-Pad4): track 0.00 -> 2.19 mm
- net GND: track 0.00 -> 1.83 mm, vias 0 -> 10
- added copper zone on B.Cu, net Earth
- added copper zone on F.Cu, net Earth
- added copper zone on In1.Cu, net Earth
- added copper zone on In2.Cu, net Earth
- added copper zone on B.Cu, net GND
- added copper zone on F.Cu, net GND
- added copper zone on In1.Cu, net GND
- added copper zone on In2.Cu, net GND
Other:
- board outline added: 146.1 x 29.9 mm
- copper layers 2 -> 4

Commit message: Routing almost finished
Parts:
- removed TP10, TP9: TestPoint, TestPoint:TestPoint_Pad_D1.0mm
- added R29: 10, Resistor_SMD:R_0603_1608Metric_Pad0.98x0.95mm_HandSolder, F.Cu at (162.6, 80.2)
- FB3: value BLM31PG601SN1L -> 100R @ 100MHz; footprint Inductor_SMD:L_1206_3216Metric -> Inductor_SMD:L_0603_1608Metric
- moved BT1 240.9 mm to (182.0, 74.5), turned to 180 degrees
- moved C27 240.1 mm to (164.4, 89.1)
- moved C29 237.9 mm to (170.8, 79.6), turned to -90 degrees
- moved C48 237.9 mm to (175.2, 82.5)
- moved C28 237.4 mm to (169.3, 78.6), turned to 90 degrees
- moved C31 236.2 mm to (166.7, 88.4), turned to 90 degrees
- moved C38 236.2 mm to (168.1, 88.4), turned to -90 degrees
- moved R18 234.1 mm to (172.8, 81.5), turned to 90 degrees
- moved C42 233.5 mm to (183.6, 81.6), turned to 90 degrees
- moved C30 233.3 mm to (163.0, 86.1)
- moved C43 231.5 mm to (183.6, 79.4), turned to -90 degrees
- moved IC8 230.8 mm to (176.7, 80.0), turned to 180 degrees
- moved L1.3 229.8 mm to (197.4, 88.8)
- moved C17 229.4 mm to (194.7, 78.6), turned to 90 degrees
- moved L1.2 229.1 mm to (197.3, 83.5)
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Connections:
- net Net-(ANODE1-Pin_1) renamed /HV/HV+_tube
- net Net-(D2-A) renamed /HV/HV+_L
- net Net-(R10-Pad1) renamed /HV/HV+_mid_meas
- FB3 pad 1: +3.3V -> Net-(U1-VDDA)
- FB3 pad 2: Net-(U1-VDDA) -> +3.3V
- U1 pad 25: /CAN_BUS/CAN_RX -> Net-(U1-PA15)
Routing:
- net +3.3V: track 0.00 -> 106.9 mm, vias 0 -> 6
- net /HV/HV+_tube: track 0.00 -> 66.2 mm
- net +5V: track 0.00 -> 58.0 mm, vias 0 -> 11
- net /MCU/EN_I_SENS: track 0.00 -> 54.1 mm, vias 0 -> 2
- net /MCU/I_SENS: track 0.00 -> 52.6 mm, vias 0 -> 2
- net /MCU/VIN_SENSE: track 0.00 -> 48.4 mm, vias 0 -> 2
- net /HV/COMP_GM: track 0.00 -> 33.8 mm, vias 0 -> 2
- net /HV/FBACK_CTRL: track 0.00 -> 26.3 mm, vias 0 -> 2
- net /CAN_BUS/CAN_STBY: track 0.00 -> 21.8 mm
- net /HV/HV_meas: track 0.00 -> 18.6 mm
- net /CAN_BUS/CAN_RX: track 0.00 -> 18.1 mm, vias 0 -> 2
- net /MCU/nRESET: track 0.00 -> 18.1 mm, vias 0 -> 2
- net /MCU/I2C1_SDA: track 0.00 -> 17.8 mm, vias 0 -> 2
- net /CAN_BUS/CAN_H: track 0.00 -> 16.6 mm, vias 0 -> 2
- net /CAN_BUS/CAN_R_CTRL: track 0.00 -> 16.1 mm, vias 0 -> 2
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- added copper zone on F.Cu, net +5V
- added copper zone on In2.Cu, net +5V
- added copper zone on F.Cu, net /MCU/VIN_SENSE
- added copper zone on F.Cu, net Net-(C18-Pad1)
- added copper zone on F.Cu, net Net-(IC1-SW)
- added copper zone on F.Cu, net Net-(IC1-VIN)

Commit message: Finished routing, needs polishing
Parts:
- moved C44 3.20 mm to (155.5, 64.9), turned to 180 degrees
- moved R26 1.39 mm to (151.2, 77.5)
- moved R25 1.15 mm to (149.0, 76.6)
- moved D6 1.12 mm to (142.9, 71.4)
- moved D7 1.12 mm to (145.2, 66.2)
- moved D8 1.12 mm to (147.4, 71.4)
- moved C37 0.63 mm to (149.4, 65.7)
- moved C33 0.51 mm to (153.7, 74.2)
- moved C36 0.50 mm to (151.2, 75.7)
- moved R22 0.33 mm to (147.5, 83.7)
- moved R15 0.32 mm to (147.1, 87.7)
- moved C20 0.22 mm to (150.9, 72.6)
- moved C15 0.20 mm to (188.6, 83.2)
- moved J2 0.17 mm to (169.9, 75.5)
- moved C34 0.11 mm to (161.4, 75.9)
Routing:
- net /MCU/VIN_SENSE: track 48.4 -> 43.8 mm
- net /CAN_BUS/CAN_STBY: track 21.8 -> 23.6 mm
- net /MCU/EN_I_SENS: track 54.1 -> 52.6 mm
- net +3.3V: track 106.9 -> 105.5 mm
- net /CAN_BUS/CAN_RX: track 18.1 -> 19.6 mm
- net /PROTECTION/V_zas: track 16.7 -> 17.9 mm
- net Net-(D6-K): track 7.83 -> 8.93 mm
- net /MCU/I_SENS: track 52.6 -> 51.5 mm
- net GND: vias 57 -> 1223

Commit message: Cleanig
Routing:
- net GND: vias 1223 -> 1202
Other:
- board size 146.1 x 29.9 mm -> 145 x 29.9 mm

Commit message: Cleaning
Parts:
- added ANODE2: Conn_01x01_Pin, Connector_PinHeader_2.00mm:PinHeader_1x01_P2.00mm_Vertical, F.Cu at (204.2, 77.1)
Connections:
- F2 pad 1: /HV/HV+_tube -> Net-(ANODE2-Pin_1)
- F2 pad 2: /HV/HV+_tube -> Net-(ANODE2-Pin_1)
Routing:
- net /HV/HV+_tube: track 66.2 -> 6.71 mm
- net Net-(ANODE2-Pin_1): track 0.00 -> 52.7 mm
- net GND: vias 1202 -> 340
Other:
- outline, holes or cut-outs redrawn

Commit message: Cleaning
Parts:
- removed ANODE2: Conn_01x01_Pin, Connector_PinHeader_2.00mm:PinHeader_1x01_P2.00mm_Vertical
- removed F2: 01020071Z, SamacSys_Parts:01020071Z
Routing:
- net Net-(ANODE2-Pin_1): track 52.7 -> 0.00 mm
Other:
- board size 145 x 29.9 mm -> 86 x 29.9 mm
