File: pcb/geiger_probe.kicad_pcb (KiCad board)
At the start: 4 copper layers, 86 x 29.9 mm, 114 parts, among them IC1 LT8606IDC#TRPBF, IC2 ATA6561-GAQW-N, IC8 MCP79410T-I_MS, J1 Conn_01x05_Socket, J2 TC2030, Q1 DMN3404L, Q2 BSS138, U1 STM32L432KCUx, U2 MCP1700x-330xxMB, U3 INA186A4IDCKR, U701 GAQY212GS, U702 GAQY212GS, Y1 32,768kHz

Commit message: Unify resistor/capacitor values and footprints, add via-in-pad DRC rule, regenerate outputs
Parts:
- C22, C34: footprint Capacitor_SMD:C_1206_3216Metric_Pad1.33x1.80mm_HandSolder -> Capacitor_SMD:C_1206_3216Metric
- C32, C33, C35, C48: footprint Capacitor_SMD:C_0603_1608Metric_Pad1.08x0.95mm_HandSolder -> Capacitor_SMD:C_0603_1608Metric
- C39: value 4.7nF -> 4.7n; footprint Capacitor_SMD:C_0603_1608Metric_Pad1.08x0.95mm_HandSolder -> Capacitor_SMD:C_0603_1608Metric
- C40, C41: value 4.7pF -> 4.7p; footprint Capacitor_SMD:C_0603_1608Metric_Pad1.08x0.95mm_HandSolder -> Capacitor_SMD:C_0603_1608Metric
- C42, C43: footprint Capacitor_SMD:C_0402_1005Metric_Pad0.74x0.62mm_HandSolder -> Capacitor_SMD:C_0402_1005Metric
- R18, R19, R20, R21, R22, R23, R24, R29, R46: footprint Resistor_SMD:R_0603_1608Metric_Pad0.98x0.95mm_HandSolder -> Resistor_SMD:R_0603_1608Metric
- R8: value 100R -> 100
Routing:
- net GND: vias 340 -> 329

Commit message: Add J1 net labels and fiducials, regenerate production outputs
- Named nets on J1 pads (schematic + PCB)
- 2 fiducials for stencil alignment (hand assembly)
- Regenerate PDFs, gerber zip, interactive BOM and 3D renders
Parts:
- added FID1: Fiducial, Fiducial:Fiducial_0.5mm_Mask1mm, F.Cu at (121.3, 89.0)
- added FID2: Fiducial, Fiducial:Fiducial_0.5mm_Mask1mm, F.Cu at (198.3, 66.2)
Routing:
- net GND: vias 329 -> 326
Other:
- board text added: "CAN H"
- board text added: "CAN L"
- board text added: "EARTH"
- board text added: "GM GND"
- board text added: "GM HV"
- board text added: "GND"
- board text added: "PRI"
- board text added: "SEC"
- board text added: "VIN"
