File: pcb/hv.kicad_sch (KiCad schematic)
At the start: 29 parts, among them Q1 DMN3404L

Commit message: Fix BOM data: correct MPNs for C16/C19, HV resistor part numbers for R9/R10/R12
Parts:
- C16: Manufacturer_Part_Number 0603N100J500CT -> (none)
- C19: Manufacturer_Part_Number CC1206KKX7RC222 -> (none)
- R10, R9: Manufacturer_Part_Number HVC1206T5005JET -> HMC1206JT500M
- R11, R13: Manufacturer_Part_Number (none) -> CRCW06031M00FKTABC
- R12: Manufacturer_Part_Number HVC1206T5005JET -> SMD1206-5M1-1%
Changed lines of the file:
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@@
 			)
 		)
-		(property "Description" "0603N100J500CT"
+		(property "Description" "Unpolarized capacitor"
 			(at 129.54 114.3 0)
 			(hide yes)
@@
 			)
 		)
-		(property "Manufacturer_Part_Number" "0603N100J500CT"
+		(property "Manufacturer_Part_Number" ""
 			(at 129.54 114.3 90)
 			(hide yes)
@@
 			)
 		)
+		(property "Manufacturer_Part_Number" "CRCW06031M00FKTABC"
+			(at 147.32 113.03 0)
+			(hide yes)
+			(show_name no)
+			(do_not_autoplace no)
+			(effects
+				(font
+					(size 1.27 1.27)
+				)
+			)
+		)
 		(pin "1"
 		)
@@
 			)
 		)
-		(property "Description" "HVC1206T5005JET"
+		(property "Description" "HMC1206JT500M"
 			(at 147.32 92.71 0)
 			(hide yes)
@@
 			)
 		)
-		(property "Manufacturer_Part_Number" "HVC1206T5005JET"
+		(property "Manufacturer_Part_Number" "HMC1206JT500M"
 			(at 147.32 92.71 0)
 			(hide yes)
@@
 			)
 		)
-		(property "Description" "CC1206KKX7RC222"
+		(property "Description" "Unpolarized capacitor"
 			(at 231.14 106.68 0)
 			(hide yes)
@@
 			)
 		)
-		(property "Manufacturer_Part_Number" "CC1206KKX7RC222"
+		(property "Manufacturer_Part_Number" ""
 			(at 231.14 106.68 0)
 			(hide yes)
@@
 			)
 		)
+		(property "Manufacturer_Part_Number" "CRCW06031M00FKTABC"
+			(at 231.14 88.9 0)
+			(hide yes)
+			(show_name no)
+			(do_not_autoplace no)
+			(effects
+				(font
+					(size 1.27 1.27)
+				)
+			)
+		)
 		(pin "1"
 		)
@@
 			)
 		)
-		(property "Description" "HVC1206T5005JET"
+		(property "Description" "SMD1206-5M1-1%"
 			(at 203.2 85.09 0)
 			(hide yes)
@@
 			)
 		)
-		(property "Manufacturer_Part_Number" "HVC1206T5005JET"
+		(property "Manufacturer_Part_Number" "SMD1206-5M1-1%"
 			(at 203.2 85.09 0)
 			(hide yes)
@@
 			)
 		)
-		(property "Description" "CC1206KKX7RC222"
+		(property "Description" "Unpolarized capacitor"
 			(at 123.19 80.01 0)
 			(hide yes)
@@
 			)
 		)
-		(property "Description" "GRM43DR7LW104KW01L"
+		(property "Description" "Unpolarized capacitor"
 			(at 130.81 80.01 0)
 			(hide yes)
@@
 			)
 		)
-		(property "Description" "HVC1206T5005JET"
+		(property "Description" "HMC1206JT500M"
 			(at 147.32 102.87 0)
 			(hide yes)
@@
 			)
 		)
-		(property "Manufacturer_Part_Number" "HVC1206T5005JET"
+		(property "Manufacturer_Part_Number" "HMC1206JT500M"
 			(at 147.32 102.87 0)
 			(hide yes)
